File: WIFI_Shield_Rev3/WIFI_Shield_Rev3/SCHEMATIC_R1.brd (EAGLE design)
At the start: 54.3 x 60.9 mm, 32 parts, among them M1 NUCLEO-L452RE, U1 APDS-9306-065, U5 ESP32-C3-WROOM-02-N4

Commit message: Arreglados los jumpers que no aparecían en el BOM. Agregados comentarios adicionales
Parts:
- added JP_C1, JP_C2, JP_C3: QPC02SXGN-RC, QPC02SXGN-RC:PLACEHOLDER
Changed lines of the file:
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@@
 <setting verticaltext="up"/>
 </settings>
-<grid distance="0.1" unitdist="mm" unit="mm" style="lines" multiple="1" display="yes" altdistance="5" altunitdist="mil" altunit="mil"/>
+<grid distance="0.2" unitdist="mm" unit="mm" style="lines" multiple="1" display="yes" altdistance="5" altunitdist="mil" altunit="mil"/>
 <layers>
 <layer number="1" name="Top" color="4" fill="1" visible="yes" active="yes"/>
-<layer number="16" name="Bottom" color="1" fill="1" visible="no" active="yes"/>
+<layer number="2" name="Route2" color="16" fill="1" visible="no" active="yes"/>
+<layer number="3" name="Route3" color="17" fill="1" visible="no" active="yes"/>
+<layer number="4" name="Route4" color="18" fill="1" visible="no" active="yes"/>
+<layer number="5" name="Route5" color="19" fill="1" visible="no" active="yes"/>
+<layer number="6" name="Route6" color="25" fill="1" visible="no" active="yes"/>
+<layer number="7" name="Route7" color="26" fill="1" visible="no" active="yes"/>
+<layer number="8" name="Route8" color="27" fill="1" visible="no" active="yes"/>
+<layer number="9" name="Route9" color="28" fill="1" visible="no" active="yes"/>
+<layer number="10" name="Route10" color="29" fill="1" visible="no" active="yes"/>
+<layer number="11" name="Route11" color="30" fill="1" visible="no" active="yes"/>
+<layer number="12" name="Route12" color="20" fill="1" visible="no" active="yes"/>
+<layer number="13" name="Route13" color="21" fill="1" visible="no" active="yes"/>
+<layer number="14" name="Route14" color="22" fill="1" visible="no" active="yes"/>
+<layer number="15" name="Route15" color="23" fill="1" visible="no" active="yes"/>
+<layer number="16" name="Bottom" color="1" fill="1" visible="yes" active="yes"/>
 <layer number="17" name="Pads" color="2" fill="1" visible="yes" active="yes"/>
 <layer number="18" name="Vias" color="2" fill="1" visible="no" active="yes"/>
 <layer number="19" name="Unrouted" color="6" fill="1" visible="yes" active="yes"/>
 <layer number="20" name="Dimension" color="24" fill="1" visible="yes" active="yes"/>
-<layer number="21" name="tPlace" color="7" fill="1" visible="no" active="yes"/>
+<layer number="21" name="tPlace" color="7" fill="1" visible="yes" active="yes"/>
 <layer number="22" name="bPlace" color="7" fill="1" visible="no" active="yes"/>
 <layer number="23" name="tOrigins" color="15" fill="1" visible="yes" active="yes"/>
@@
 <element name="JP1" library="pinhead edit" package="1X03" package3d_urn="urn:adsk.eagle:package:22458/2" value="QPC02SXGN-RC" x="61.5" y="42.5" smashed="yes" rot="R270">
 <attribute name="NAME" x="59.5" y="38.5" size="1.27" layer="25" ratio="10" rot="R90"/>
-<attribute name="PARTNO" value="QPC02SXGN-RC" x="61.5" y="42.5" size="1.778" layer="27" rot="R270" display="off"/>
 <attribute name="POPULARITY" value="92" x="61.5" y="42.5" size="1.778" layer="27" rot="R270" display="off"/>
 </element>
 <element name="JP2" library="pinhead edit" package="1X03" package3d_urn="urn:adsk.eagle:package:22458/2" value="QPC02SXGN-RC" x="56" y="42.5" smashed="yes" rot="R90">
 <attribute name="NAME" x="54" y="38.5" size="1.27" layer="25" ratio="10" rot="R90"/>
-<attribute name="PARTNO" value="QPC02SXGN-RC" x="56" y="42.5" size="1.778" layer="27" rot="R90" display="off"/>
 <attribute name="POPULARITY" value="92" x="56" y="42.5" size="1.778" layer="27" rot="R90" display="off"/>
 </element>
 <element name="JP3" library="pinhead edit" package="1X03" package3d_urn="urn:adsk.eagle:package:22458/2" value="QPC02SXGN-RC" x="50.5" y="42.5" smashed="yes" rot="R90">
 <attribute name="NAME" x="48.5" y="38.5" size="1.27" layer="25" ratio="10" rot="R90"/>
-<attribute name="PARTNO" value="QPC02SXGN-RC" x="50.5" y="42.5" size="1.778" layer="27" rot="R90" display="off"/>
 <attribute name="POPULARITY" value="92" x="50.5" y="42.5" size="1.778" layer="27" rot="R90" display="off"/>
 </element>
+<element name="JP_C1" library="QPC02SXGN-RC" package="PLACEHOLDER" value="QPC02SXGN-RC" x="22.5" y="71.6" smashed="yes">
+<attribute name="PARTNO" value="QPC02SXGN-RC" x="22.5" y="71.6" size="1.778" layer="27" display="off"/>
+</element>
+<element name="JP_C2" library="QPC02SXGN-RC" package="PLACEHOLDER" value="QPC02SXGN-RC" x="22.5" y="68.9" smashed="yes">
+<attribute name="PARTNO" value="QPC02SXGN-RC" x="22.5" y="68.9" size="1.778" layer="27" display="off"/>
+</element>
+<element name="JP_C3" library="QPC02SXGN-RC" package="PLACEHOLDER" value="QPC02SXGN-RC" x="22.5" y="66.2" smashed="yes">
+<attribute name="PARTNO" value="QPC02SXGN-RC" x="22.5" y="66.2" size="1.778" layer="27" display="off"/>
+</element>
 </elements>
